File: kicad/doorbell.kicad_sch (KiCad schematic)
At the start: 112 parts, among them J1 USB-C (USB4105), J2 WF26 bus, J3 USB-JST, K1 GAQW212GS, K2 GAQY212GS, K3 GAQY412EH, K4 GAQY412EH, K5 G6K-2F-Y DC12, K6 GAQY412EH, Q3 AO3400A, Q4 AO3400A, SW1 BOOT, SW2 EN, SW3 Tueroeffner (door release), SW4 Sprechen/Hoeren (talk), U1 ESP32-S3-WROOM-1U-N16R8, U2 SGM2212-3.3, U3 ES8311, U4 LP5907MFX-3.3

Commit message: hardware: finalize JST service inlet
Parts:
- removed D4: SS14, PCM_JLCPCB:D_SMA, symbol PCM_JLCPCB-Diodes:Schottky,SS14
- removed J1: USB-C (USB4105), Connector_USB:USB_C_Receptacle_GCT_USB4105-xx-A_16P_TopMnt_Horizontal, symbol Connector:USB_C_Receptacle_USB2.0_16P
- removed R13, R14: 5.1k, PCM_JLCPCB:R_0603, symbol PCM_JLCPCB-Resistors:0603,5.1kΩ
- renumbered D15 to D4, J3 to J1
Connections:
- net WALL_VBUS_IN is gone; now on net VBUS: D4.2, J1.1 (Pin_1)
- net STATUS_LED: now also U1.7 (IO7); no longer U1.22 (IO14)
- net VBUS: no longer D4.1, F1.1
- new net VBUS_PROTECTED: D4.1, F1.1
- no-connect marks 24 -> 22
Other:
- note added: "USB"
- note removed: "USB-C"
- moved on the sheet: C22, D10, D4, F1, J1
